File: PiHAT.sch (KiCad schematic (older format))
At the start: 17 parts, among them U1 LM2596T-ADJ

Commit message: Add files via upload
Parts:
- removed Cff: 5nF, symbol Device:CP1_Small
- removed D1: 1N5822, Diode_THT:D_DO-201AD_P15.24mm_Horizontal, symbol Diode:1N5822
- removed R1: 1.0k, symbol Device:R
- removed R2: 3.1k, symbol Device:R
- removed R5, R6: 1M, symbol Device:R
- removed U?: MCP3008, symbol Analog_ADC:MCP3008
- added D?: 1N5821, Diode_THT:D_DO-201AD_P15.24mm_Horizontal, symbol Diode:1N5821
- added J1, J2, J? (x4): B8B-EH-A, SHDR8W64P0X250_1X8_2250X380X600P, symbol SamacSys_Parts:B8B-EH-A
- added J? (x6): XT30UPB-M, SHDR2W160P0X500_1X2_1020X520X1070P, symbol XT30UPB-M:XT30UPB-M
- added J?: B3B-ZR__LF__SN_, SHDR3W50P0X150_1X3_600X350X450P, symbol B3B-ZR__LF__SN_:B3B-ZR__LF__SN_
- Cin: value 100uF -> 680uF
Connections:
- net +5V: now also J?.1
- net +6V: now also J?.1, J?.1, J?.1, J?.1
- net GND: now also U?.1 (A0), U?.2 (A1), U?.24 (A5), U?.3 (A2), U?.4 (A3), U?.5 (A4), D?.2 (A), J?.2, J?.2, J?.2, J?.2, J?.2, J?.2
- net P26: now reaches U?.1 (I3)
- net P26: now also J2.4
- net P1: now reaches U?.10 (S1)
- net P1: now also J?.10 (GPIO15/RXD), U?.10 (S1); no longer J?.38 (GPIO20/MOSI1)
- net P0: now reaches U?.11 (S0)
- net P0: now also J?.8 (GPIO14/TXD), U?.11 (S0); no longer J?.35 (GPIO19/MISO1)
- net P30: now reaches U?.12 (I7)
- net P30: now also J2.8
- net P29: now reaches U?.13 (I6)
- net P29: now also J2.7
- net P28: now reaches U?.14 (I5)
- net P28: now also J2.6
- net P27: now reaches U?.15 (I4)
- net P27: now also J2.5
- net P25: now reaches U?.2 (I2)
- net P25: now also J2.3
- net P24: now reaches U?.3 (I1)
- net P24: now also J2.2
- net P23: now reaches U?.4 (I0)
- net P23: now also J2.1
- net P6: now reaches U?.5 (Z)
- net P6: now also J?.40 (GPIO21/SCLK1); no longer J?.16 (GPIO23)
- net P44: now reaches U?.6 (~Z)
- net P44: now also J?.6
- net P5: now reaches U?.7 (~E)
- net P5: now also J?.38 (GPIO20/MOSI1); no longer J?.15 (GPIO22)
- net P2: now reaches U?.9 (S2)
- net P2: now also J?.36 (GPIO16), U?.9 (S2); no longer J?.40 (GPIO21/SCLK1)
- net P18: now reaches U?.1 (I3)
- net P18: now also J1.4
- net P22: now reaches U?.12 (I7)
- net P22: now also J1.8
- net P21: now reaches U?.13 (I6)
- net P21: now also J1.7
- net P20: now reaches U?.14 (I5)
- net P20: now also J1.6
- net P19: now reaches U?.15 (I4)
- net P19: now also J1.5
- net P17: now reaches U?.2 (I2)
- net P17: now also J1.3
- net P16: now reaches U?.3 (I1)
- net P16: now also J1.2
- net P4: now reaches U?.5 (Z)
- net P4: now also J?.35 (GPIO19/MISO1); no longer J?.12 (GPIO18/PWM0)
- net P43: now reaches U?.6 (~Z)
- net P43: now also J?.5
- net P3: now reaches J?.11 (GPIO17), U?.7 (~E)
- net +3V3: now reaches J?.1 (3V3)
- net +3V3: now also J?.17 (3V3), J?.1
- net P33: now reaches J?.13 (GPIO27)
- net P33: now also J?.3
- net P9: now reaches J?.18 (GPIO24)
- net P9: now also J?.2
- net P39: now reaches J?.19 (MOSI0/GPIO10)
- net P39: now also J?.1
- net at Cout.1, J?.2 (5V), L1.1: now also U1.4 (FB)
- net P38: now reaches J?.21 (MISO0/GPIO9)
- net P38: now also J?.8
- net P31: now reaches J?.22 (GPIO25)
- net P31: now also J?.1
- net P40: now reaches J?.23 (SCLK0/GPIO11)
- net P40: now also J?.2
- net P37: now reaches J?.24 (~CE0~/GPIO8)
- net P37: now also J?.7
- net P36: now reaches J?.26 (~CE1~/GPIO7)
- net P36: now also J?.6
- net P34: now reaches J?.27 (ID_SD/GPIO0)
- net P34: now also J?.4
- net P35: now reaches J?.28 (ID_SC/GPIO1)
- net P35: now also J?.5
- net P10: now reaches J?.29 (GCLK1/GPIO5)
- net P10: now also J?.3
- net P12: now reaches J?.3 (SDA/GPIO2), U?.27 (SDA)
- net P14: now reaches J?.31 (GCLK2/GPIO6), U?.23 (~OE)
- net P41: now reaches J?.32 (PWM0/GPIO12)
- net P41: now also J?.3
- net P42: now reaches J?.33 (PWM1/GPIO13)
- net P42: now also J?.4
- net P32: now reaches J?.37 (GPIO26)
- net P32: now also J?.2
- net P11: now reaches J?.5 (SCL/GPIO3), U?.26 (SCL)
- net P13: now reaches J?.7 (GCLK0/GPIO4), U?.25 (EXTCLK)
- net at L1.2, U1.2 (OUT): now also D?.1 (K)
- net P15: now reaches R3.1
- net P15: now also J1.1
- net at U?.10 (LED4): now also J?.5
- net at U?.11 (LED5): now also J?.6
- net at U?.12 (LED6): now also J?.7
- net at U?.13 (LED7): now also J?.8
- net at U?.15 (LED8): now also J?.1
- net at U?.16 (LED9): now also J?.2
- net at U?.17 (LED10): now also J?.3
- net at U?.18 (LED11): now also J?.4
- net at U?.19 (LED12): now also J?.5
- net at U?.20 (LED13): now also J?.6
- net at U?.21 (LED14): now also J?.7
- net at U?.22 (LED15): now also J?.8
- net at U?.6 (LED0): now also J?.1
- net at U?.7 (LED1): now also J?.2
- net at U?.8 (LED2): now also J?.3
- net at U?.9 (LED3): now also J?.4
- new net P45: J?.12 (GPIO18/PWM0), J?.7
- new net P7: J?.15 (GPIO22), J?.8
- new net P8: J?.1, J?.16 (GPIO23)
Other:
- moved on the sheet: R3

Commit message: Add files via upload
Parts:
- added R3, R5: 1.3k, symbol Device:R
- added R4, R6: 4.3k, symbol Device:R
- gave numbers to parts that had none: 16
- renumbered Cin to Cin1, Cout to Cout1, R3 to R1, R4 to R2, U1 to U3
Connections:
- net GND: now also R4.2, R6.2
- net P4: now also R5.1, R6.1; no longer U4.5 (Z)
- net P6: now also R3.1, R4.1; no longer U1.5 (Z)
- new net: R3.2, U1.5 (Z)
- new net: R5.2, U4.5 (Z)

Commit message: Add files via upload
Parts:
- removed J4: Raspberry_Pi_2_3, symbol Connector:Raspberry_Pi_2_3
- added J15: Conn_02x20_Odd_Even, RPi_Hat:Pin_Header_Straight_2x20, symbol Connector_Generic:Conn_02x20_Odd_Even
- Cin1: footprint (none) -> Capacitor_SMD:CP_Elec_4x5.8
- Cout1: footprint (none) -> Capacitor_SMD:CP_Elec_4x5.4
- J1, J14, J2, J3, J5, J6: footprint SHDR8W64P0X250_1X8_2250X380X600P -> SamacSys_Parts:SHDR8W64P0X250_1X8_2250X380X600P
- J10, J11, J12, J7, J8, J9: footprint SHDR2W160P0X500_1X2_1020X520X1070P -> SamacSys_Parts:SHDR2W160P0X500_1X2_1020X520X1070P
- J13: footprint SHDR3W50P0X150_1X3_600X350X450P -> SamacSys_Parts:SHDR3W50P0X150_1X3_600X350X450P
- L1: footprint (none) -> Inductor_SMD:L_12x12mm_H8mm
- R1, R2, R3, R4, R5, R6: footprint (none) -> Resistor_SMD:R_0402_1005Metric
- U1, U4: footprint (none) -> Mux:SOIC127P600X175-16N
Connections:
- net +3V3: now also J15.1 (Pin_1), J15.17 (Pin_17)
- net +5V: now also J15.4 (Pin_4)
- net GND: now also J15.14 (Pin_14), J15.20 (Pin_20), J15.25 (Pin_25), J15.30 (Pin_30), J15.34 (Pin_34), J15.39 (Pin_39), J15.6 (Pin_6), J15.9 (Pin_9)
- net P0: now also J15.8 (Pin_8)
- net P1: now also J15.10 (Pin_10)
- net P10: now also J15.29 (Pin_29)
- net P11: now also J15.5 (Pin_5)
- net P12: now also J15.3 (Pin_3)
- net P13: now also J15.7 (Pin_7)
- net P14: now also J15.31 (Pin_31)
- net P2: now also J15.36 (Pin_36)
- net P3: now also J15.11 (Pin_11)
- net P31: now also J15.22 (Pin_22)
- net P32: now also J15.37 (Pin_37)
- net P33: now also J15.13 (Pin_13)
- net P34: now also J15.27 (Pin_27)
- net P35: now also J15.28 (Pin_28)
- net P36: now also J15.26 (Pin_26)
- net P37: now also J15.24 (Pin_24)
- net P38: now also J15.21 (Pin_21)
- net P39: now also J15.19 (Pin_19)
- net P4: now also J15.35 (Pin_35)
- net P40: now also J15.23 (Pin_23)
- net P41: now also J15.32 (Pin_32)
- net P42: now also J15.33 (Pin_33)
- net P45: now also J15.12 (Pin_12)
- net P5: now also J15.38 (Pin_38)
- net P6: now also J15.40 (Pin_40)
- net P7: now also J15.15 (Pin_15)
- net P8: now also J15.16 (Pin_16)
- net P9: now also J15.18 (Pin_18)
- net 46: now reaches Cout1.1, L1.1, U3.4 (FB)
- net 46: now also J15.2 (Pin_2)

Commit message: Add files via upload
Connections:
- net +3V3: now also J15.18 (Pin_18), J15.2 (Pin_2); no longer J15.1 (Pin_1), J15.17 (Pin_17)
- net +5V: now also J15.3 (Pin_3); no longer J15.4 (Pin_4)
- net 46: now also J15.1 (Pin_1); no longer J15.2 (Pin_2)
- net GND: now also J15.10 (Pin_10), J15.13 (Pin_13), J15.19 (Pin_19), J15.26 (Pin_26), J15.29 (Pin_29), J15.33 (Pin_33), J15.40 (Pin_40), J15.5 (Pin_5); no longer J15.14 (Pin_14), J15.20 (Pin_20), J15.25 (Pin_25), J15.30 (Pin_30), J15.34 (Pin_34), J15.39 (Pin_39), J15.6 (Pin_6), J15.9 (Pin_9)
- net P0: now also J15.7 (Pin_7), U1.7 (~E); no longer J15.8 (Pin_8), U1.11 (S0), U4.11 (S0)
- net P1: now also J15.9 (Pin_9), U1.9 (S2), U4.9 (S2); no longer J15.10 (Pin_10), U1.10 (S1), U4.10 (S1)
- net P10: now also J15.30 (Pin_30); no longer J15.29 (Pin_29)
- net P11: now also J15.6 (Pin_6); no longer J15.5 (Pin_5)
- net P12: now also J15.4 (Pin_4); no longer J15.3 (Pin_3)
- net P13: now also J15.8 (Pin_8); no longer J15.7 (Pin_7)
- net P14: now also J15.32 (Pin_32); no longer J15.31 (Pin_31)
- net P2: now also J15.35 (Pin_35), U1.10 (S1), U4.10 (S1); no longer J15.36 (Pin_36), U1.9 (S2), U4.9 (S2)
- net P23: now also J2.4; no longer J2.1
- net P24: now also J2.3; no longer J2.2
- net P25: now also J2.2; no longer J2.3
- net P26: now also J2.1; no longer J2.4
- net P3: now also J15.12 (Pin_12); no longer J15.11 (Pin_11)
- net P31: now also J15.21 (Pin_21); no longer J15.22 (Pin_22)
- net P32: now also J15.38 (Pin_38); no longer J15.37 (Pin_37)
- net P33: now also J15.14 (Pin_14); no longer J15.13 (Pin_13)
- net P34: now also J15.28 (Pin_28); no longer J15.27 (Pin_27)
- net P35: now also J15.27 (Pin_27); no longer J15.28 (Pin_28)
- net P36: now also J15.25 (Pin_25); no longer J15.26 (Pin_26)
- net P37: now also J15.23 (Pin_23); no longer J15.24 (Pin_24)
- net P38: now also J15.22 (Pin_22); no longer J15.21 (Pin_21)
- net P39: now also J15.20 (Pin_20); no longer J15.19 (Pin_19)
- net P4: now also J15.36 (Pin_36); no longer J15.35 (Pin_35)
- net P40: now also J15.24 (Pin_24); no longer J15.23 (Pin_23)
- net P41: now also J15.31 (Pin_31); no longer J15.32 (Pin_32)
- net P42: now also J15.34 (Pin_34); no longer J15.33 (Pin_33)
- net P45: now also J15.11 (Pin_11); no longer J15.12 (Pin_12)
- net P5: now also J15.37 (Pin_37), U1.11 (S0), U4.11 (S0); no longer J15.38 (Pin_38), U1.7 (~E)
- net P6: now also J15.39 (Pin_39); no longer J15.40 (Pin_40)
- net P7: now also J15.16 (Pin_16); no longer J15.15 (Pin_15)
- net P8: now also J15.15 (Pin_15); no longer J15.16 (Pin_16)
- net P9: now also J15.17 (Pin_17); no longer J15.18 (Pin_18)

Commit message: Add files via upload
Parts:
- removed Cout1: 220uF, Capacitor_SMD:CP_Elec_4x5.4, symbol Device:CP1_Small
- removed J10, J11, J12, J7, J8, J9: XT30UPB-M, SamacSys_Parts:SHDR2W160P0X500_1X2_1020X520X1070P, symbol XT30UPB-M:XT30UPB-M
- removed J13: B3B-ZR__LF__SN_, SamacSys_Parts:SHDR3W50P0X150_1X3_600X350X450P, symbol B3B-ZR__LF__SN_:B3B-ZR__LF__SN_
- removed U2: PCA9685PW, Package_SO:TSSOP-28_4.4x9.7mm_P0.65mm, symbol Driver_LED:PCA9685PW
- removed U3: LM2596T-ADJ, Package_TO_SOT_THT:TO-220-5_P3.4x3.7mm_StaggerOdd_Lead3.8mm_Vertical, symbol Regulator_Switching:LM2596T-ADJ
- added Cout1: EEEFK1A221AL, Cap:CAP_EEEFK1A221AL, symbol EEEFK1A221AL:EEEFK1A221AL
- added J10, J11, J12, J16, J7, J8, J9: B2B-PH-K-S(LF)(SN), B2B:JST_B2B-PH-K-S(LF)(SN), symbol B2B-PH-K-S_LF__SN_:B2B-PH-K-S(LF)(SN)
- added J13: B4B-PH-K-S(LF)(SN), B4B:JST_B4B-PH-K-S(LF)(SN), symbol B4B-PH-K-S_LF__SN_:B4B-PH-K-S(LF)(SN)
- added U2: PCA9552PW,118, PCA9552PW:SOP65P640X110-24N, symbol PCA9552PW_118:PCA9552PW,118
- added U3: LM2596S-5, Package_TO_SOT_SMD:TO-263-5_TabPin3, symbol Regulator_Switching:LM2596S-5
- Cin1: footprint Capacitor_SMD:CP_Elec_4x5.8 -> Capacitor_SMD:CP_Elec_10x10.5
Connections:
- net +3V3: now also J16.1
- net +5V: now also J10.1, J11.1, J12.1, U2.24 (VDD)
- net +6V: now also J7.1, J9.1; no longer Cin1.1
- net 46: now also Cout1.1, U3.4 (FB)
- net GND: now also Cout1.2, J10.2, J11.2, J12.2, J16.2, J7.2, J8.2, J9.2, U2.1 (A0), U2.12 (VSS), U2.2 (A1), U2.3 (A2), U3.3 (GND), U3.5 (~ON~/OFF)
- net P10: now also J3.7
- net P11: now also U2.22 (SCL)
- net P12: now also U2.23 (SDA)
- net P13: now also J14.1
- net P14: now also U2.21 (~RESET)
- net P31: now also J14.8; no longer J3.1
- net P32: now also J13.2; no longer J3.2
- net P33: now also J14.3; no longer J3.3
- net P34: now also J3.6; no longer J3.4
- net P36: now also J3.4; no longer J3.6
- net P37: now also J3.2; no longer J3.7
- net P38: now also J3.1; no longer J3.8
- net P39: now also J14.7; no longer J14.1
- net P40: now also J3.3; no longer J14.2
- net P41: now also J3.8; no longer J14.3
- net P42: now also J13.1; no longer J14.4
- net P43: now also J13.4; no longer J14.5
- net P44: now also J13.3; no longer J14.6
- net P45: now also J14.2; no longer J14.7
- net P7: now also J14.5; no longer J14.8
- net P8: now also J14.4
- net P9: now also J14.6
- net at D1.1 (K), L1.2: now also U3.2 (OUT)
- net at J5.5: now also U2.8 (LED4)
- net at J5.6: now also U2.9 (LED5)
- net at J5.7: now also U2.10 (LED6)
- net at J5.8: now also U2.11 (LED7)
- net at J6.1: now also U2.13 (LED8)
- net at J6.2: now also U2.14 (LED9)
- net at J6.3: now also U2.15 (LED10)
- net at J6.4: now also U2.16 (LED11)
- net at J6.5: now also U2.17 (LED12)
- net at J6.6: now also U2.18 (LED13)
- net at J6.7: now also U2.19 (LED14)
- net at J6.8: now also U2.20 (LED15)
- net at J5.1: now also U2.4 (LED0)
- net at J5.2: now also U2.5 (LED1)
- net at J5.3: now also U2.6 (LED2)
- net at J5.4: now also U2.7 (LED3)
- new net +8V: Cin1.1, J8.1, U3.1 (VIN)
