File: PiHAT.kicad_pcb (KiCad board)
At the start: 2 copper layers, 0 parts

Commit message: Add files via upload
Parts:
- added ?: , RPi_Hat:RPi_Hat_Mounting_Hole, F.Cu at (130.8, 21.6)
- added Cin1: 680uF, Capacitor_SMD:CP_Elec_4x5.8, F.Cu at (73.6, 19.7)
- added Cout1: 220uF, Capacitor_SMD:CP_Elec_4x5.4, F.Cu at (47.2, 23.0)
- added D1: 1N5821, Diode_THT:D_DO-201AD_P15.24mm_Horizontal, F.Cu at (22.2, 16.7)
- added J1: B8B-EH-A, SamacSys_Parts:SHDR8W64P0X250_1X8_2250X380X600P, F.Cu at (23.1, 0.21)
- added J10: XT30UPB-M, SamacSys_Parts:SHDR2W160P0X500_1X2_1020X520X1070P, F.Cu at (34.9, 23.4)
- added J11: XT30UPB-M, SamacSys_Parts:SHDR2W160P0X500_1X2_1020X520X1070P, F.Cu at (47.2, 5.96)
- added J12: XT30UPB-M, SamacSys_Parts:SHDR2W160P0X500_1X2_1020X520X1070P, F.Cu at (54.9, 12.7)
- added J13: B3B-ZR__LF__SN_, SamacSys_Parts:SHDR3W50P0X150_1X3_600X350X450P, F.Cu at (82.7, 20.4)
- added J14: B8B-EH-A, SamacSys_Parts:SHDR8W64P0X250_1X8_2250X380X600P, F.Cu at (23.1, 10.9)
- added J15: Conn_02x20_Odd_Even, RPi_Hat:Pin_Header_Straight_2x20, F.Cu at (159.9, 166.0)
- added J2: B8B-EH-A, SamacSys_Parts:SHDR8W64P0X250_1X8_2250X380X600P, F.Cu at (47.1, -5.14)
- added J3: B8B-EH-A, SamacSys_Parts:SHDR8W64P0X250_1X8_2250X380X600P, F.Cu at (23.1, 5.56)
- added J5: B8B-EH-A, SamacSys_Parts:SHDR8W64P0X250_1X8_2250X380X600P, F.Cu at (47.1, 0.21)
- added J6: B8B-EH-A, SamacSys_Parts:SHDR8W64P0X250_1X8_2250X380X600P, F.Cu at (23.1, -5.14)
- added J7: XT30UPB-M, SamacSys_Parts:SHDR2W160P0X500_1X2_1020X520X1070P, F.Cu at (59.0, 5.96)
- added J8: XT30UPB-M, SamacSys_Parts:SHDR2W160P0X500_1X2_1020X520X1070P, F.Cu at (23.2, 23.4)
- added J9: XT30UPB-M, SamacSys_Parts:SHDR2W160P0X500_1X2_1020X520X1070P, F.Cu at (43.2, 16.7)
- added L1: 33uH, Inductor_SMD:L_12x12mm_H8mm, F.Cu at (75.3, -0.99)
- added R1: 1k, Resistor_SMD:R_0402_1005Metric, F.Cu at (21.3, 27.8)
- added R2: 2k, Resistor_SMD:R_0402_1005Metric, F.Cu at (24.2, 27.8)
- added R3: 1.3k, Resistor_SMD:R_0402_1005Metric, F.Cu at (27.1, 27.8)
- added R4: 4.3k, Resistor_SMD:R_0402_1005Metric, F.Cu at (30.0, 27.8)
- added R5: 1.3k, Resistor_SMD:R_0402_1005Metric, F.Cu at (32.9, 27.8)
- added R6: 4.3k, Resistor_SMD:R_0402_1005Metric, F.Cu at (35.8, 27.8)
- added U1: 74LS151, Mux:SOIC127P600X175-16N, F.Cu at (56.4, 21.8)
- added U2: PCA9685PW, Package_SO:TSSOP-28_4.4x9.7mm_P0.65mm, F.Cu at (83.3, 11.8)
- added U3: LM2596T-ADJ, Package_TO_SOT_THT:TO-220-5_P3.4x3.7mm_StaggerOdd_Lead3.8mm_Vertical, F.Cu at (69.7, 15.1)
- added U4: 74LS151, Mux:SOIC127P600X175-16N, F.Cu at (65.5, 22.5)
Routing:
- net (no net): vias 0 -> 4

Commit message: Add files via upload
Parts:
- added ?: , RPi_Hat:RPi_Hat_Mounting_Hole, F.Cu at (103.9, 93.5)
- added ?: , RPi_Hat:RPi_Hat_Mounting_Hole, F.Cu at (45.9, 44.5)
- added ?: , RPi_Hat:RPi_Hat_Mounting_Hole, F.Cu at (45.9, 93.5)
- added REF**: CAMERA_HOLE, RPi_Hat:CAMERA_HOLE, F.Cu at (87.6, 85.0)
- Cin1, Cout1, D1, J15, L1, U3: moved to B.Cu
- moved J15 148.3 mm to (74.9, 44.5), turned to 270 degrees
- moved J1 84.2 mm to (68.6, 71.1)
- moved L1 82.3 mm to (74.9, 81.3), turned to 270 degrees
- moved J10 81.8 mm to (-19.7, 84.4)
- moved J11 81.8 mm to (-7.36, 66.9)
- moved J12 81.8 mm to (0.33, 73.7)
- moved J14 81.8 mm to (-31.5, 71.9)
- moved J3 81.8 mm to (-31.5, 66.5)
- moved J7 81.8 mm to (4.39, 66.9)
- moved J9 81.8 mm to (-11.4, 77.6)
- moved J13 81.8 mm to (28.1, 81.3)
- moved D1 81.3 mm to (82.5, 71.1), turned to 180 degrees
- moved J2 76.2 mm to (92.7, 55.9)
- moved R2 73.3 mm to (60.5, 91.4), turned to 270 degrees
- moved R1 71.6 mm to (60.6, 87.6), turned to 270 degrees
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Connections:
- J15 pad 1: +3V3 -> 46
- J15 pad 10: P1 -> GND
- J15 pad 11: P3 -> P45
- J15 pad 12: P45 -> P3
- J15 pad 13: P33 -> GND
- J15 pad 14: GND -> P33
- J15 pad 15: P7 -> P8
- J15 pad 16: P8 -> P7
- J15 pad 17: +3V3 -> P9
- J15 pad 18: P9 -> +3V3
- J15 pad 19: P39 -> GND
- J15 pad 2: 46 -> +3V3
- J15 pad 20: GND -> P39
- J15 pad 21: P38 -> P31
- J15 pad 22: P31 -> P38
- J15 pad 23: P40 -> P37
- J15 pad 24: P37 -> P40
- J15 pad 25: GND -> P36
- J15 pad 26: P36 -> GND
- J15 pad 27: P34 -> P35
- J15 pad 28: P35 -> P34
- J15 pad 29: P10 -> GND
- J15 pad 3: P12 -> +5V
- J15 pad 30: GND -> P10
- J15 pad 31: P14 -> P41
- J15 pad 32: P41 -> P14
- J15 pad 33: P42 -> GND
- J15 pad 34: GND -> P42
- J15 pad 35: P4 -> P2
- J15 pad 36: P2 -> P4
- J15 pad 37: P32 -> P5
- J15 pad 38: P5 -> P32
- J15 pad 39: GND -> P6
- J15 pad 4: +5V -> P12
- J15 pad 40: P6 -> GND
- J15 pad 5: P11 -> GND
- J15 pad 6: GND -> P11
- J15 pad 7: P13 -> P0
- J15 pad 8: P0 -> P13
- J15 pad 9: GND -> P1
- J2 pad 1: P23 -> P26
- J2 pad 2: P24 -> P25
- J2 pad 3: P25 -> P24
- J2 pad 4: P26 -> P23
- U1 pad 10: P1 -> P2
- U1 pad 11: P0 -> P5
- U1 pad 7: P5 -> P0
- U1 pad 9: P2 -> P1
- U4 pad 10: P1 -> P2
- U4 pad 11: P0 -> P5
- U4 pad 9: P2 -> P1
Routing:
- net P1: track 0.00 -> 147.8 mm, vias 0 -> 3
- net GND: track 0.00 -> 139.0 mm, vias 0 -> 3
- net P5: track 0.00 -> 118.7 mm, vias 0 -> 3
- net P0: track 0.00 -> 118.6 mm, vias 0 -> 1
- net P2: track 0.00 -> 116.7 mm, vias 0 -> 3
- net P11: track 0.00 -> 95.3 mm, vias 0 -> 1
- net P6: track 0.00 -> 65.7 mm, vias 0 -> 1
- net P14: track 0.00 -> 57.0 mm, vias 0 -> 1
- net P3: track 0.00 -> 55.6 mm, vias 0 -> 1
- net Net-(D1-Pad1): track 0.00 -> 38.5 mm
- net P23: track 0.00 -> 31.6 mm
- net P13: track 0.00 -> 31.3 mm, vias 0 -> 1
- net P24: track 0.00 -> 27.4 mm
- net P30: track 0.00 -> 26.7 mm
- net P16: track 0.00 -> 25.1 mm
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
Commit message: Add files via upload
Parts:
- added J16: B2B-PH-K-S(LF)(SN), B2B:JST_B2B-PH-K-S(LF)(SN), F.Cu at (111.8, 83.8)
- Cin1: footprint Capacitor_SMD:CP_Elec_4x5.8 -> Capacitor_SMD:CP_Elec_10x10.5
- Cout1: value 220uF -> EEEFK1A221AL; footprint Capacitor_SMD:CP_Elec_4x5.4 -> Cap:CAP_EEEFK1A221AL
- J10, J11, J12, J7, J8, J9: value XT30UPB-M -> B2B-PH-K-S(LF)(SN); footprint SamacSys_Parts:SHDR2W160P0X500_1X2_1020X520X1070P -> B2B:JST_B2B-PH-K-S(LF)(SN)
- J13: value B3B-ZR__LF__SN_ -> B4B-PH-K-S(LF)(SN); footprint SamacSys_Parts:SHDR3W50P0X150_1X3_600X350X450P -> B4B:JST_B4B-PH-K-S(LF)(SN)
- U2: value PCA9685PW -> PCA9552PW,118; footprint Package_SO:TSSOP-28_4.4x9.7mm_P0.65mm -> PCA9552PW:SOP65P640X110-24N
- U3: value LM2596T-ADJ -> LM2596S-5; footprint Package_TO_SOT_THT:TO-220-5_P3.4x3.7mm_StaggerOdd_Lead3.8mm_Vertical -> Package_TO_SOT_SMD:TO-263-5_TabPin3
- moved J9 123.4 mm to (111.8, 71.1)
- moved J10 120.0 mm to (100.3, 83.8), turned to 180 degrees
- moved J3 112.1 mm to (76.2, 35.6)
- moved J7 107.9 mm to (111.8, 77.5)
- moved J11 107.8 mm to (100.3, 71.1), turned to 180 degrees
- moved J12 100.1 mm to (100.3, 77.5), turned to 180 degrees
- moved J14 91.1 mm to (52.1, 35.6)
- moved J13 87.0 mm to (102.0, 35.4), turned to 180 degrees
- moved U3 6.04 mm to (51.8, 84.1), turned to 180 degrees
- moved D1 3.81 mm to (82.5, 67.3)
- moved L1 3.81 mm to (78.7, 81.3)
- moved R4 2.77 mm to (76.2, 58.4), turned to 90 degrees
- moved Cout1 2.55 mm to (66.0, 83.8)
- moved Cin1 2.54 mm to (58.4, 72.4)
- moved J8 2.46 mm to (58.4, 74.9), turned to 180 degrees
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Connections:
- Cin1 pad 1: +6V -> +8V
- J10 pad 1: +6V -> +5V
- J12 pad 1: +3V3 -> +5V
- J13 pad 1: P8 -> P42
- J13 pad 2: P9 -> P32
- J13 pad 3: P10 -> P44
- J14 pad 1: P39 -> P13
- J14 pad 2: P40 -> P45
- J14 pad 3: P41 -> P33
- J14 pad 4: P42 -> P8
- J14 pad 5: P43 -> P7
- J14 pad 6: P44 -> P9
- J14 pad 7: P45 -> P39
- J14 pad 8: P7 -> P31
- J3 pad 1: P31 -> P38
- J3 pad 2: P32 -> P37
- J3 pad 3: P33 -> P40
- J3 pad 4: P34 -> P36
- J3 pad 6: P36 -> P34
- J3 pad 7: P37 -> P10
- J3 pad 8: P38 -> P41
- J8 pad 1: +6V -> +8V
- U2 pad 10: Net-(J5-Pad5) -> Net-(J5-Pad7)
- U2 pad 11: Net-(J5-Pad6) -> Net-(J5-Pad8)
- U2 pad 12: Net-(J5-Pad7) -> GND
- U2 pad 13: Net-(J5-Pad8) -> Net-(J6-Pad1)
- U2 pad 14: GND -> Net-(J6-Pad2)
- U2 pad 15: Net-(J6-Pad1) -> Net-(J6-Pad3)
- U2 pad 16: Net-(J6-Pad2) -> Net-(J6-Pad4)
- U2 pad 17: Net-(J6-Pad3) -> Net-(J6-Pad5)
- U2 pad 18: Net-(J6-Pad4) -> Net-(J6-Pad6)
- U2 pad 19: Net-(J6-Pad5) -> Net-(J6-Pad7)
- U2 pad 20: Net-(J6-Pad6) -> Net-(J6-Pad8)
- U2 pad 21: Net-(J6-Pad7) -> P14
- U2 pad 22: Net-(J6-Pad8) -> P11
- U2 pad 23: P14 -> P12
- U2 pad 24: GND -> +5V
- U2 pad 4: GND -> Net-(J5-Pad1)
- U2 pad 5: GND -> Net-(J5-Pad2)
- U2 pad 6: Net-(J5-Pad1) -> Net-(J5-Pad3)
- U2 pad 7: Net-(J5-Pad2) -> Net-(J5-Pad4)
- U2 pad 8: Net-(J5-Pad3) -> Net-(J5-Pad5)
- U2 pad 9: Net-(J5-Pad4) -> Net-(J5-Pad6)
- U3 pad 1: +6V -> +8V
Routing:
- net +5V: track 5.98 -> 155.4 mm, vias 2 -> 8
- net +3V3: track 0.00 -> 135.2 mm
- net GND: track 139.0 -> 242.9 mm, vias 3 -> 11
- net 46: track 17.8 -> 117.4 mm
- net P43: track 0.00 -> 94.1 mm, vias 0 -> 1
- net P4: track 1.52 -> 68.4 mm, vias 0 -> 1
- net P44: track 0.00 -> 37.7 mm, vias 0 -> 1
- net Net-(D1-Pad1): track 38.5 -> 64.2 mm
- net P13: track 31.3 -> 12.8 mm, vias 1 -> 0
- net P33: track 0.00 -> 14.2 mm
- net P42: track 0.00 -> 14.1 mm
- net P7: track 0.00 -> 14.1 mm
- net P32: track 0.00 -> 14.0 mm
- net P34: track 0.00 -> 13.3 mm
- net P45: track 0.00 -> 12.8 mm
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- added copper zone on B.Cu, net (none)
- added copper zone on F.Cu, net GND
Other:
- board outline added: 78.7 x 66 mm
- board text added: "Raspberry Pi CAP 2021"

Commit message: Add files via upload
Parts:
- removed REF**: CAMERA_HOLE, RPi_Hat:CAMERA_HOLE
Routing:
- net P2: track 116.3 -> 117.2 mm
Other:
- outline, holes or cut-outs redrawn
